Commit message: 模型里imu修改和相机相关joint名称修改

File: src/tiangong2pro_urdf/urdf/tiangong2.0_pro_urdf.urdf (robot description, URDF)
Before this commit: robot tiangong2pro_urdf, 37 links, 36 joints
Links:
- removed link camera_body_back_link
- removed link camera_body_front_link
- removed link camera_head_link
- removed link imu_link
- added link imu, mass 0.02; collision mesh filename=package://tiangong2pro_urdf/meshes/imu_link.STL; visual mesh filename=package://tiangong2pro_urdf/meshes/imu_link.STL
- added link ob_camera_back_link, mass 0.1; collision mesh filename=package://tiangong2pro_urdf/meshes/camera_body_back_link.STL; visual mesh filename=package://tiangong2pro_urdf/meshes/camera_body_back_link.STL
- added link ob_camera_head_link, mass 0.1; collision mesh filename=package://tiangong2pro_urdf/meshes/camera_head_link.STL; visual mesh filename=package://tiangong2pro_urdf/meshes/camera_head_link.STL
- added link ob_camera_waist_link, mass 0.1; collision mesh filename=package://tiangong2pro_urdf/meshes/camera_body_front_link.S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; visual mesh filename=package://tiangong2pro_urdf/meshes/camera_body_front_link.S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
Joints:
- joint camera_body_back_joint: child camera_body_back_link -> ob_camera_back_link
- joint camera_body_front_joint: child camera_body_front_link -> ob_camera_waist_link
- joint camera_head_joint: child camera_head_link -> ob_camera_head_link
- joint imu_joint: child imu_link -> imu

File: src/tiangong2pro_urdf/urdf/tiangong2.0_pro_with_hands.urdf (robot description, URDF)
Before this commit: robot tiangong2pro_urdf_with_hands, 63 links, 62 joints
Links:
- removed link camera_body_back_link
- removed link camera_body_front_link
- removed link camera_head_link
- removed link imu_link
- added link imu, mass 0.02; collision mesh filename=package://tiangong2pro_urdf/meshes/imu_link.STL; visual mesh filename=package://tiangong2pro_urdf/meshes/imu_link.STL
- added link ob_camera_back_link, mass 0.1; collision mesh filename=package://tiangong2pro_urdf/meshes/camera_body_back_link.STL; visual mesh filename=package://tiangong2pro_urdf/meshes/camera_body_back_link.STL
- added link ob_camera_head_link, mass 0.1; collision mesh filename=package://tiangong2pro_urdf/meshes/camera_head_link.STL; visual mesh filename=package://tiangong2pro_urdf/meshes/camera_head_link.STL
- added link ob_camera_waist_link, mass 0.1; collision mesh filename=package://tiangong2pro_urdf/meshes/camera_body_front_link.S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; visual mesh filename=package://tiangong2pro_urdf/meshes/camera_body_front_link.S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
Joints:
- joint camera_body_back_joint: child camera_body_back_link -> ob_camera_back_link
- joint camera_body_front_joint: child camera_body_front_link -> ob_camera_waist_link
- joint camera_head_joint: child camera_head_link -> ob_camera_head_link
- joint imu_joint: child imu_link -> imu
